File: Version 1.2 - Copy.kicad_pcb (KiCad board)
At the start: 4 copper layers, 40 x 40 mm, 39 parts, among them J2 Conn_01x02_Pin, J3 Conn_01x12_Socket, J4 Conn_01x16_Socket, J4 Conn_Coaxial, U1 BGA2801, U2 BGA420, U3 AS179-92LF, U4 SX1278, U5 74LVC1G19, Y1 ECS-TXO-2520-33-400-AN-TR

Commit message: Ordered Version
Routing:
- net GND: track 31.2 -> 32.6 mm
- net /TCXO_OUT: track 4.26 -> 4.82 mm
Other:
- board text added: "WIT PICO COM BOARD V1.0"
- board text removed: "WIT PICO COM BOARD V0"
